File: pcb/fpga.kicad_sch (KiCad schematic)
At the start: 31 parts

Commit message: added new_vga and sram
Parts:
- C? (x24): value (none) -> ~
Other:
- added sheet sram (sram.kicad_sch)
- added sheet vga (vga.kicad_sch)
Changed lines of the file:
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@@
       (effects (font (size 1.27 1.27)) (justify left))
     )
-    (property "Value" "" (id 1) (at 88.9 124.46 0)
+    (property "Value" "~" (id 1) (at 88.9 124.46 0)
       (effects (font (size 1.27 1.27)) (justify left))
     )
@@
       (effects (font (size 1.27 1.27)) hide)
     )
-    (property "Value" "" (id 1) (at 34.29 173.99 0))
+    (property "Value" "~" (id 1) (at 34.29 173.99 0))
     (property "Footprint" "" (id 2) (at 34.29 179.07 0)
       (effects (font (size 1.27 1.27)) hide)
@@
       (effects (font (size 1.27 1.27)) (justify left))
     )
-    (property "Value" "" (id 1) (at 134.62 124.46 0)
+    (property "Value" "~" (id 1) (at 134.62 124.46 0)
       (effects (font (size 1.27 1.27)) (justify left))
     )
@@
       (effects (font (size 1.27 1.27)) (justify left))
     )
-    (property "Value" "" (id 1) (at 50.8 124.46 0)
+    (property "Value" "~" (id 1) (at 50.8 124.46 0)
       (effects (font (size 1.27 1.27)) (justify left))
     )
@@
       (effects (font (size 1.27 1.27)) (justify left))
     )
-    (property "Value" "" (id 1) (at 50.8 154.94 0)
+    (property "Value" "~" (id 1) (at 50.8 154.94 0)
       (effects (font (size 1.27 1.27)) (justify left))
     )
@@
       (effects (font (size 1.27 1.27)) (justify left))
     )
-    (property "Value" "" (id 1) (at 142.24 124.46 0)
+    (property "Value" "~" (id 1) (at 142.24 124.46 0)
       (effects (font (size 1.27 1.27)) (justify left))
     )
@@
       (effects (font (size 1.27 1.27)) hide)
     )
-    (property "Value" "" (id 1) (at 34.29 113.03 0))
+    (property "Value" "~" (id 1) (at 34.29 113.03 0))
     (property "Footprint" "" (id 2) (at 34.29 118.11 0)
       (effects (font (size 1.27 1.27)) hide)
@@
       (effects (font (size 1.27 1.27)) (justify left))
     )
-    (property "Value" "" (id 1) (at 73.66 124.46 0)
+    (property "Value" "~" (id 1) (at 73.66 124.46 0)
       (effects (font (size 1.27 1.27)) (justify left))
     )
@@
       (effects (font (size 1.27 1.27)) (justify left))
     )
-    (property "Value" "" (id 1) (at 50.8 185.42 0)
+    (property "Value" "~" (id 1) (at 50.8 185.42 0)
       (effects (font (size 1.27 1.27)) (justify left))
     )
@@
       (effects (font (size 1.27 1.27)) (justify left))
     )
-    (property "Value" "" (id 1) (at 66.04 185.42 0)
+    (property "Value" "~" (id 1) (at 66.04 185.42 0)
       (effects (font (size 1.27 1.27)) (justify left))
     )
@@
       (effects (font (size 1.27 1.27)) (justify left))
     )
-    (property "Value" "" (id 1) (at 96.52 124.46 0)
+    (property "Value" "~" (id 1) (at 96.52 124.46 0)
       (effects (font (size 1.27 1.27)) (justify left))
     )
@@
       (effects (font (size 1.27 1.27)) (justify left))
     )
-    (property "Value" "" (id 1) (at 58.42 124.46 0)
+    (property "Value" "~" (id 1) (at 58.42 124.46 0)
       (effects (font (size 1.27 1.27)) (justify left))
     )
@@
       (effects (font (size 1.27 1.27)) (justify left))
     )
-    (property "Value" "" (id 1) (at 66.04 124.46 0)
+    (property "Value" "~" (id 1) (at 66.04 124.46 0)
       (effects (font (size 1.27 1.27)) (justify left))
     )
@@
       (effects (font (size 1.27 1.27)) hide)
     )
-    (property "Value" "" (id 1) (at 34.29 130.81 0))
+    (property "Value" "~" (id 1) (at 34.29 130.81 0))
     (property "Footprint" "" (id 2) (at 34.29 125.73 0)
       (effects (font (size 1.27 1.27)) hide)
@@
       (effects (font (size 1.27 1.27)) (justify left))
     )
-    (property "Value" "" (id 1) (at 73.66 185.42 0)
+    (property "Value" "~" (id 1) (at 73.66 185.42 0)
       (effects (font (size 1.27 1.27)) (justify left))
     )
@@
       (effects (font (size 1.27 1.27)) (justify left))
     )
-    (property "Value" "" (id 1) (at 111.76 124.46 0)
+    (property "Value" "~" (id 1) (at 111.76 124.46 0)
       (effects (font (size 1.27 1.27)) (justify left))
     )
@@
       (effects (font (size 1.27 1.27)) (justify left))
     )
-    (property "Value" "" (id 1) (at 81.28 124.46 0)
+    (property "Value" "~" (id 1) (at 81.28 124.46 0)
       (effects (font (size 1.27 1.27)) (justify left))
     )
@@
       (effects (font (size 1.27 1.27)) (justify left))
     )
-    (property "Value" "" (id 1) (at 43.18 124.46 0)
+    (property "Value" "~" (id 1) (at 43.18 124.46 0)
       (effects (font (size 1.27 1.27)) (justify left))
     )
@@
       (effects (font (size 1.27 1.27)) (justify left))
     )
-    (property "Value" "" (id 1) (at 73.66 154.94 0)
+    (property "Value" "~" (id 1) (at 73.66 154.94 0)
       (effects (font (size 1.27 1.27)) (justify left))
     )
@@
       (effects (font (size 1.27 1.27)) (justify left))
     )
-    (property "Value" "" (id 1) (at 119.38 124.46 0)
+    (property "Value" "~" (id 1) (at 119.38 124.46 0)
       (effects (font (size 1.27 1.27)) (justify left))
     )
@@
       (effects (font (size 1.27 1.27)) (justify left))
     )
-    (property "Value" "" (id 1) (at 35.56 124.46 0)
+    (property "Value" "~" (id 1) (at 35.56 124.46 0)
       (effects (font (size 1.27 1.27)) (justify left))
     )
@@
       (effects (font (size 1.27 1.27)) (justify left))
     )
-    (property "Value" "" (id 1) (at 127 124.46 0)
+    (property "Value" "~" (id 1) (at 127 124.46 0)
       (effects (font (size 1.27 1.27)) (justify left))
     )
@@
       (effects (font (size 1.27 1.27)) (justify left))
     )
-    (property "Value" "" (id 1) (at 58.42 185.42 0)
+    (property "Value" "~" (id 1) (at 58.42 185.42 0)
       (effects (font (size 1.27 1.27)) (justify left))
     )
@@
       (effects (font (size 1.27 1.27)) (justify left))
     )
-    (property "Value" "" (id 1) (at 104.14 124.46 0)
+    (property "Value" "~" (id 1) (at 104.14 124.46 0)
       (effects (font (size 1.27 1.27)) (justify left))
     )
@@
       (effects (font (size 1.27 1.27)) (justify left))
     )
-    (property "Value" "" (id 1) (at 81.28 185.42 0)
+    (property "Value" "~" (id 1) (at 81.28 185.42 0)
       (effects (font (size 1.27 1.27)) (justify left))
     )
@@
       (effects (font (size 1.27 1.27)) (justify left))
     )
-    (property "Value" "" (id 1) (at 43.18 185.42 0)
+    (property "Value" "~" (id 1) (at 43.18 185.42 0)
       (effects (font (size 1.27 1.27)) (justify left))
     )
@@
       (effects (font (size 1.27 1.27)) (justify left))
     )
-    (property "Value" "" (id 1) (at 110.49 154.94 0)
+    (property "Value" "~" (id 1) (at 110.49 154.94 0)
       (effects (font (size 1.27 1.27)) (justify left))
     )
@@
     )
   )
+  (sheet (at 35.56 82.55) (size 25.4 13.97) (fields_autoplaced)
+    (stroke (width 0.1524) (type solid) (color 0 0 0 0))
+    (fill (color 0 0 0 0.0000))
+    (property "Sheet name" "vga" (id 0) (at 35.56 81.8384 0)
+      (effects (font (size 1.27 1.27)) (justify left bottom))
+    )
+    (property "Sheet file" "vga.kicad_sch" (id 1) (at 35.56 97.1046 0)
+      (effects (font (size 1.27 1.27)) (justify left top))
+    )
+  )
   (sheet (at 127 43.18) (size 26.67 25.4) (fields_autoplaced)
     (stroke (width 0.1524) (type solid) (color 0 0 0 0))
@@
       (effects (font (size 1.27 1.27)) (justify left top))
     )
+  )
+  (sheet (at 76.2 83.82) (size 26.67 13.97) (fields_autoplaced)
+    (stroke (width 0.1524) (type solid) (color 0 0 0 0))
+    (fill (color 0 0 0 0.0000))
+    (property "Sheet name" "sram" (id 0) (at 76.2 83.1084 0)
+      (effects (font (size 1.27 1.27)) (justify left bottom))
+    )
+    (property "Sheet file" "sram.kicad_sch" (id 1) (at 76.2 98.3746 0)
+      (effects (font (size 1.27 1.27)) (justify left top))
+    )

Commit message: commit before merge
Parts:
- removed C? (x6): ~, symbol Device:C
- removed C?: 47u, Capacitor_SMD:C_0805_2012Metric_Pad1.18x1.45mm_HandSolder, symbol Device:C

Commit message: maybe finished schematic
Parts:
- added D? (x4): LED, LED_SMD:LED_1206_3216Metric_Pad1.42x1.75mm_HandSolder, symbol Device:LED
- added R? (x4): 330, Resistor_SMD:R_2512_6332Metric_Pad1.40x3.35mm_HandSolder, symbol Device:R
- C? (x10): value ~ -> 470n
- C? (x7): value ~ -> 4.7u
- C?: value ~ -> 330
Connections:
- net GND: now also R?.2, R?.2, R?.2, R?.2
- new net: D?.1 (K), R?.1 (x4)
- new net FPGA_DEBUG_LED_BLOCK14_1: D?.2 (A)
- new net FPGA_DEBUG_LED_BLOCK15_1: D?.2 (A)
- new net FPGA_DEBUG_LED_BLOCK35_1: D?.2 (A)
- new net FPGA_DEBUG_LED_BLOCK35_2: D?.2 (A)
Other:
- note added: "FPGA DEBUG LEDS"
- note added: "FPGA MCU SPI"
- note added: "FPGA Programming signals"
- note added: "GPIO / MCU SPI"
- note added: "VGA / SRAM"
- note removed: "FPGA JTAG Debug"
- note removed: "TODO: * UG483: 7 Series FPGAs PCB Design Guide ▶ Information about decoupling capacitors * XAPP586: Using SPI Flash with 7 Series FPGAs ▶ How to connect the Flash chip and JTAG connector"
- moved on the sheet: C?
