File: pcb/mcu.kicad_sch (KiCad schematic)
At the start: 8 parts

Commit message: kicad said I needed to save
Parts:
- J?: value 1658525-9 -> (none); footprint 1658525-9-ribbon:TE_1658525-9 -> (none)
- U? (x2): footprint mcu_kicad:EFM32GG990F1024 -> BGA112
Changed lines of the file:
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@@
       (effects (font (size 1.524 1.524)))
     )
-    (property "Footprint" "mcu_kicad:EFM32GG990F1024" (id 2) (at 217.17 45.974 0)
+    (property "Footprint" "BGA112" (id 2) (at 217.17 45.974 0)
       (effects (font (size 1.524 1.524)) hide)
     )
@@
       (effects (font (size 1.524 1.524)))
     )
-    (property "Footprint" "mcu_kicad:EFM32GG990F1024" (id 2) (at 74.93 42.164 0)
+    (property "Footprint" "BGA112" (id 2) (at 74.93 42.164 0)
       (effects (font (size 1.524 1.524)) hide)
     )
@@
     (in_bom yes) (on_board yes)
     (property "Reference" "J?" (id 0) (at 262.89 179.07 0))
-    (property "Value" "1658525-9" (id 1) (at 262.89 147.32 0))
-    (property "Footprint" "1658525-9-ribbon:TE_1658525-9" (id 2) (at 262.89 162.56 0)
+    (property "Value" "" (id 1) (at 262.89 147.32 0))
+    (property "Footprint" "" (id 2) (at 262.89 162.56 0)
       (effects (font (size 1.27 1.27)) (justify left bottom) hide)
     )

Commit message: add spi pins and finish onboard_controller
Parts:
- J?: value (none) -> 1658525-9; footprint (none) -> 1658525-9-ribbon:TE_1658525-9
Connections:
- net GND: now also C?.2
- net js_gpio_1: now also U?.J3 (PD15); no longer U?.J1 (PC1)
- net mcu_spi_output: now reaches U?.H1 (PC0)
- net mcu_spi_clock: now reaches U?.K1 (PB7)
- net mcu_spi_chip_select: now reaches U?.L1 (PB8)
- new net mcu_spi_input: U?.J1 (PC1)
Other:
- note added: "Spi mcu <-> fpga"
Changed lines of the file:
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@@
+    (stroke (width 0) (type default) (color 0 0 0 0))
+  )
+  (polyline (pts (xy 15.24 176.53) (xy 64.77 176.53))
     (stroke (width 0) (type default) (color 0 0 0 0))
   )
@@
     (stroke (width 0) (type default) (color 0 0 0 0))
   )
+  (polyline (pts (xy 64.77 176.53) (xy 64.77 142.24))
+    (stroke (width 0) (type default) (color 0 0 0 0))
+  )
   (wire (pts (xy 137.16 74.93) (xy 137.16 77.47))
     (stroke (width 0) (type default) (color 0 0 0 0))
@@
     (stroke (width 0) (type default) (color 0 0 0 0))
   )
+  (polyline (pts (xy 15.24 142.24) (xy 15.24 176.53))
+    (stroke (width 0) (type default) (color 0 0 0 0))
+  )
   (wire (pts (xy 247.65 69.85) (xy 247.65 72.39))
     (stroke (width 0) (type default) (color 0 0 0 0))
   )
+  (polyline (pts (xy 15.24 142.24) (xy 64.77 142.24))
+    (stroke (width 0) (type default) (color 0 0 0 0))
+  )
   (wire (pts (xy 137.16 68.58) (xy 142.24 68.58))
     (stroke (width 0) (type default) (color 0 0 0 0))
@@
   (wire (pts (xy 113.03 119.38) (xy 119.38 119.38))
     (stroke (width 0) (type default) (color 0 0 0 0))
+  )
+  (text "Spi mcu <-> fpga" (at 29.21 146.05 0)
+    (effects (font (size 1.27 1.27)) (justify left bottom))
   )
   (label "må vi spesifisere noe her?" (at 113.03 123.19 0)
@@
     )
   )
+  (global_label "mcu_spi_chip_select" (shape bidirectional) (at 45.72 157.48 0) (fields_autoplaced)
+    (effects (font (size 1 1)) (justify left))
+    (property "Intersheet References" "${INTERSHEET_REFS}" (id 0) (at 62.8105 157.4175 0)
+      (effects (font (size 1 1)) (justify left) hide)
+    )
+  )
   (global_label "con_js_vert_1" (shape bidirectional) (at 250.19 165.1 180) (fields_autoplaced)
     (effects (font (size 0.5 0.5)) (justify right))
@@
     (property "Intersheet References" "${INTERSHEET_REFS}" (id 0) (at 242.2257 64.7388 0)
       (effects (font (size 0.5 0.5)) (justify left) hide)
+    )
+  )
+  (global_label "mcu_spi_chip_select" (shape bidirectional) (at 237.49 82.55 0) (fields_autoplaced)
+    (effects (font (size 1 1)) (justify left))
+    (property "Intersheet References" "${INTERSHEET_REFS}" (id 0) (at 254.5805 82.4875 0)
+      (effects (font (size 1 1)) (justify left) hide)
     )
   )
@@
     )
   )
+  (global_label "js_gpio_1" (shape bidirectional) (at 186.69 110.49 180) (fields_autoplaced)
+    (effects (font (size 0.8 0.8)) (justify right))
+    (property "Intersheet References" "${INTERSHEET_REFS}" (id 0) (at 179.6081 110.44 0)
+      (effects (font (size 0.8 0.8)) (justify right) hide)
+    )
+  )
   (global_label "bo_button_4" (shape bidirectional) (at 44.45 86.36 180) (fields_autoplaced)
     (effects (font (size 0.5 0.5)) (justify right))
@@
     )
   )
+  (global_label "mcu_spi_clock" (shape bidirectional) (at 237.49 52.07 0) (fields_autoplaced)
+    (effects (font (size 1 1)) (justify left))
+    (property "Intersheet References" "${INTERSHEET_REFS}" (id 0) (at 250.1519 52.0075 0)
+      (effects (font (size 1 1)) (justify left) hide)
+    )
+  )
   (global_label "mcu_serial_clock" (shape bidirectional) (at 152.4 64.77 0) (fields_autoplaced)
     (effects (font (size 0.5 0.5)) (justify left))
@@
     (property "Intersheet References" "${INTERSHEET_REFS}" (id 0) (at 244.121 162.5288 0)
       (effects (font (size 0.5 0.5)) (justify right) hide)
+    )
+  )
+  (global_label "mcu_spi_input" (shape bidirectional) (at 186.69 105.41 180) (fields_autoplaced)
+    (effects (font (size 1 1)) (justify right))
+    (property "Intersheet References" "${INTERSHEET_REFS}" (id 0) (at 174.2186 105.3475 0)
+      (effects (font (size 1 1)) (justify right) hide)
     )
   )
@@
     )
   )
+  (global_label "mcu_spi_output" (shape bidirectional) (at 45.72 161.29 0) (fields_autoplaced)
+    (effects (font (size 1 1)) (justify left))
+    (property "Intersheet References" "${INTERSHEET_REFS}" (id 0) (at 59.1914 161.2275 0)
+      (effects (font (size 1 1)) (justify left) hide)
+    )
+  )
+  (global_label "mcu_spi_output" (shape bidirectional) (at 186.69 74.93 180) (fields_autoplaced)
+    (effects (font (size 1 1)) (justify right))
+    (property "Intersheet References" "${INTERSHEET_REFS}" (id 0) (at 173.2186 74.8675 0)
+      (effects (font (size 1 1)) (justify right) hide)
+    )
+  )
   (global_label "bo_js_hor_1" (shape bidirectional) (at 186.69 100.33 180) (fields_autoplaced)
     (effects (font (size 1 1)) (justify right))
@@
     )
   )
+  (global_label "mcu_spi_clock" (shape bidirectional) (at 45.72 153.67 0) (fields_autoplaced)
+    (effects (font (size 1 1)) (justify left))
+    (property "Intersheet References" "${INTERSHEET_REFS}" (id 0) (at 58.3819 153.6075 0)
+      (effects (font (size 1 1)) (justify left) hide)
+    )
+  )
   (global_label "con_hor_1" (shape bidirectional) (at 237.49 113.03 0) (fields_autoplaced)
     (effects (font (size 0.5 0.5)) (justify left))
@@
     )
   )
-  (global_label "js_gpio_1" (shape bidirectional) (at 186.69 105.41 180) (fields_autoplaced)
-    (effects (font (size 0.8 0.8)) (justify right))
-    (property "Intersheet References" "${INTERSHEET_REFS}" (id 0) (at 179.6081 105.36 0)
-      (effects (font (size 0.8 0.8)) (justify right) hide)
-    )
-  )
   (global_label "mcu_serial_out" (shape bidirectional) (at 152.4 66.04 0) (fields_autoplaced)
     (effects (font (size 0.5 0.5)) (justify left))
@@
     (property "Intersheet References" "${INTERSHEET_REFS}" (id 0) (at 179.6081 123.14 0)
       (effects (font (size 0.8 0.8)) (justify right) hide)
+    )
+  )
+  (global_label "mcu_spi_input" (shape bidirectional) (at 45.72 167.64 0) (fields_autoplaced)
+    (effects (font (size 1 1)) (justify left))
+    (property "Intersheet References" "${INTERSHEET_REFS}" (id 0) (at 58.1914 167.5775 0)
+      (effects (font (size 1 1)) (justify left) hide)
     )
   )
@@
     (in_bom yes) (on_board yes)
     (property "Reference" "J?" (id 0) (at 262.89 179.07 0))
-    (property "Value" "" (id 1) (at 262.89 147.32 0))
-    (property "Footprint" "" (id 2) (at 262.89 162.56 0)
+    (property "Value" "1658525-9" (id 1) (at 262.89 147.32 0))
+    (property "Footprint" "1658525-9-ribbon:TE_1658525-9" (id 2) (at 262.89 162.56 0)
       (effects (font (size 1.27 1.27)) (justify left bottom) hide)
     )
@@
       (effects (font (size 1.27 1.27)) hide)
     )
+    (pin "1")
+  )
+  (symbol (lib_id "power:GND") (at 113.03 132.08 0) (unit 1)
+    (in_bom yes) (on_board yes) (fields_autoplaced)
+    (property "Reference" "#PWR?" (id 0) (at 113.03 138.43 0)
+      (effects (font (size 1.27 1.27)) hide)
+    )
+    (property "Value" "GND" (id 1) (at 113.03 137.16 0))
+    (property "Footprint" "" (id 2) (at 113.03 132.08 0)
+      (effects (font (size 1.27 1.27)) hide)
+    )
+    (property "Datasheet" "" (id 3) (at 113.03 132.08 0)
+      (effects (font (size 1.27 1.27)) hide)
+    )
