File: pcb/psu.kicad_sch (KiCad schematic)
At the start: 32 parts

Commit message: maybe finished schematic
Parts:
- added JP? (x3): Jumper_2_Open, symbol Jumper:Jumper_2_Open
Connections:
- net +1V0: now also JP?.2 (B); no longer C?.1, C?.1, L?.2, R?.1, U?.1 (VO)
- net +1V8: now also JP?.1 (A); no longer C?.1, C?.1, L?.1, R?.1
- net +3V3: now also JP?.2 (B); no longer C?.1, C?.1, L?.2, R?.1
- new net: C?.1, C?.1, JP?.1 (A), L?.2, R?.1, U?.1 (VO)
- new net: C?.1, C?.1, JP?.2 (B), L?.1, R?.1
- new net: C?.1, C?.1, JP?.1 (A), L?.2, R?.1
- no-connect marks 0 -> 1
Other:
- note added: "lp>3.5A, lrms>3.1A"
Changed lines of the file:
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@@
   (junction (at 71.12 49.53) (diameter 0) (color 0 0 0 0)
   )
+  (no_connect (at 177.8 134.62))
   (wire (pts (xy 64.135 82.55) (xy 71.12 82.55))
     (stroke (width 0) (type default) (color 0 0 0 0))
@@
     (stroke (width 0) (type default) (color 0 0 0 0))
   )
+  (wire (pts (xy 248.92 49.53) (xy 255.905 49.53))
+    (stroke (width 0) (type default) (color 0 0 0 0))
+  )
   (wire (pts (xy 127 134.62) (xy 130.81 134.62))
     (stroke (width 0) (type default) (color 0 0 0 0))
@@
     (stroke (width 0) (type default) (color 0 0 0 0))
   )
+  (wire (pts (xy 275.59 134.62) (xy 270.51 134.62))
+    (stroke (width 0) (type default) (color 0 0 0 0))
+  )
   (wire (pts (xy 154.94 158.75) (xy 154.94 163.83))
     (stroke (width 0) (type default) (color 0 0 0 0))
@@
     (stroke (width 0) (type default) (color 0 0 0 0))
   )
-  (wire (pts (xy 26.67 134.62) (xy 26.67 133.35))
+  (wire (pts (xy 16.51 134.62) (xy 21.59 134.62))
     (stroke (width 0) (type default) (color 0 0 0 0))
   )
@@
     (stroke (width 0) (type default) (color 0 0 0 0))
   )
-  (wire (pts (xy 35.56 134.62) (xy 26.67 134.62))
-    (stroke (width 0) (type default) (color 0 0 0 0))
-  )
   (wire (pts (xy 106.68 124.46) (xy 106.68 125.73))
     (stroke (width 0) (type default) (color 0 0 0 0))
@@
     (stroke (width 0) (type default) (color 0 0 0 0))
   )
+  (wire (pts (xy 260.35 134.62) (xy 254 134.62))
+    (stroke (width 0) (type default) (color 0 0 0 0))
+  )
   (wire (pts (xy 91.44 158.75) (xy 130.81 158.75))
     (stroke (width 0) (type default) (color 0 0 0 0))
@@
     (stroke (width 0) (type default) (color 0 0 0 0))
   )
-  (wire (pts (xy 232.41 49.53) (xy 255.905 49.53))
+  (wire (pts (xy 232.41 49.53) (xy 238.76 49.53))
     (stroke (width 0) (type default) (color 0 0 0 0))
   )
@@
     (stroke (width 0) (type default) (color 0 0 0 0))
   )
+  (wire (pts (xy 31.75 134.62) (xy 35.56 134.62))
+    (stroke (width 0) (type default) (color 0 0 0 0))
+  )
   (wire (pts (xy 115.57 62.23) (xy 111.76 62.23))
     (stroke (width 0) (type default) (color 0 0 0 0))
@@
   (wire (pts (xy 182.88 100.33) (xy 119.38 100.33))
     (stroke (width 0) (type default) (color 0 0 0 0))
+  )
+  (text "lp>3.5A, lrms>3.1A" (at 234.95 41.91 0)
+    (effects (font (size 1.27 1.27)) (justify left bottom))
   )
   (text "4.5V - 18V\n" (at 35.56 53.34 0)
@@
     (pin "2")
   )
-  (symbol (lib_id "power:+3V3") (at 254 134.62 0) (unit 1)
+  (symbol (lib_id "power:+3V3") (at 275.59 134.62 0) (unit 1)
     (in_bom yes) (on_board yes) (fields_autoplaced)
-    (property "Reference" "#PWR?" (id 0) (at 254 138.43 0)
-      (effects (font (size 1.27 1.27)) hide)
-    )
-    (property "Value" "+3V3" (id 1) (at 254 129.54 0))
-    (property "Footprint" "" (id 2) (at 254 134.62 0)
-      (effects (font (size 1.27 1.27)) hide)
-    )
-    (property "Datasheet" "" (id 3) (at 254 134.62 0)
+    (property "Reference" "#PWR?" (id 0) (at 275.59 138.43 0)
+      (effects (font (size 1.27 1.27)) hide)
+    )
+    (property "Value" "+3V3" (id 1) (at 275.59 129.54 0))
+    (property "Footprint" "" (id 2) (at 275.59 134.62 0)
+      (effects (font (size 1.27 1.27)) hide)
+    )
+    (property "Datasheet" "" (id 3) (at 275.59 134.62 0)
       (effects (font (size 1.27 1.27)) hide)
     )
@@
     )
     (property "Datasheet" "~" (id 3) (at 193.04 129.54 0)
+      (effects (font (size 1.27 1.27)) hide)
+    )
+    (pin "1")
+    (pin "2")
+  )
+  (symbol (lib_id "Jumper:Jumper_2_Open") (at 26.67 134.62 0) (unit 1)
+    (in_bom yes) (on_board yes) (fields_autoplaced)
+    (property "Reference" "JP?" (id 0) (at 26.67 128.27 0))
+    (property "Value" "Jumper_2_Open" (id 1) (at 26.67 130.81 0))
+    (property "Footprint" "" (id 2) (at 26.67 134.62 0)
+      (effects (font (size 1.27 1.27)) hide)
+    )
+    (property "Datasheet" "~" (id 3) (at 26.67 134.62 0)
       (effects (font (size 1.27 1.27)) hide)
     )
@@
     (pin "1")
   )
+  (symbol (lib_id "Jumper:Jumper_2_Open") (at 243.84 49.53 0) (unit 1)
+    (in_bom yes) (on_board yes) (fields_autoplaced)
+    (property "Reference" "JP?" (id 0) (at 243.84 43.18 0))
+    (property "Value" "Jumper_2_Open" (id 1) (at 243.84 45.72 0))
+    (property "Footprint" "" (id 2) (at 243.84 49.53 0)
+      (effects (font (size 1.27 1.27)) hide)
+    )
+    (property "Datasheet" "~" (id 3) (at 243.84 49.53 0)
+      (effects (font (size 1.27 1.27)) hide)
+    )
+    (pin "1")
+    (pin "2")
+  )
   (symbol (lib_id "Device:C") (at 106.68 71.12 0) (unit 1)
     (in_bom yes) (on_board yes)
@@
     )
     (property "Datasheet" "~" (id 3) (at 214.63 124.46 0)
+      (effects (font (size 1.27 1.27)) hide)
+    )
+    (pin "1")
+    (pin "2")
+  )
+  (symbol (lib_id "Jumper:Jumper_2_Open") (at 265.43 134.62 0) (unit 1)
+    (in_bom yes) (on_board yes) (fields_autoplaced)
+    (property "Reference" "JP?" (id 0) (at 265.43 128.27 0))
+    (property "Value" "Jumper_2_Open" (id 1) (at 265.43 130.81 0))
+    (property "Footprint" "" (id 2) (at 265.43 134.62 0)
+      (effects (font (size 1.27 1.27)) hide)
+    )
+    (property "Datasheet" "~" (id 3) (at 265.43 134.62 0)
       (effects (font (size 1.27 1.27)) hide)
     )
@@
     (pin "2")
   )
-  (symbol (lib_id "power:+1V8") (at 26.67 133.35 0) (unit 1)
+  (symbol (lib_id "power:+1V8") (at 16.51 134.62 0) (unit 1)
     (in_bom yes) (on_board yes) (fields_autoplaced)
-    (property "Reference" "#PWR?" (id 0) (at 26.67 137.16 0)
-      (effects (font (size 1.27 1.27)) hide)
-    )
-    (property "Value" "+1V8" (id 1) (at 26.67 128.27 0))
-    (property "Footprint" "" (id 2) (at 26.67 133.35 0)
-      (effects (font (size 1.27 1.27)) hide)
-    )
-    (property "Datasheet" "" (id 3) (at 26.67 133.35 0)
-      (effects (font (size 1.27 1.27)) hide)
-    )
+    (property "Reference" "#PWR?" (id 0) (at 16.51 138.43 0)
+      (effects (font (size 1.27 1.27)) hide)
+    )
+    (property "Value" "+1V8" (id 1) (at 16.51 129.54 0))
+    (property "Footprint" "" (id 2) (at 16.51 134.62 0)
+      (effects (font (size 1.27 1.27)) hide)
+    )
+    (property "Datasheet" "" (id 3) (at 16.51 134.62 0)
+      (effects (font (size 1.27 1.27)) hide)
+    )
