File: pcb/onboard_controller.kicad_sch (KiCad schematic)
At the start: 13 parts

Commit message: add footprints
Parts:
- R401, R402, R403, R404, R405, R406: renamed from R?; footprint (none) -> Resistor_SMD:R_0805_2012Metric_Pad1.20x1.40mm_HandSolder
- gave numbers to parts that had none: 7
Changed lines of the file:
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@@
   (symbol (lib_id "dk_Pushbutton-Switches:GPTS203211B") (at 140.97 69.85 0) (unit 1)
     (in_bom yes) (on_board yes) (fields_autoplaced)
-    (property "Reference" "S?" (id 0) (at 140.97 62.23 0))
+    (property "Reference" "S404" (id 0) (at 140.97 62.23 0))
     (property "Value" "GPTS203211B" (id 1) (at 140.97 64.77 0))
     (property "Footprint" "digikey-footprints:PushButton_12x12mm_THT_GPTS203211B" (id 2) (at 146.05 64.77 0)
@@
   (symbol (lib_id "COM-09032:COM-09032") (at 55.88 38.1 0) (unit 1)
     (in_bom yes) (on_board yes) (fields_autoplaced)
-    (property "Reference" "U?" (id 0) (at 64.77 38.0999 0)
+    (property "Reference" "U401" (id 0) (at 64.77 38.0999 0)
       (effects (font (size 1.27 1.27)) (justify left))
     )
@@
   (symbol (lib_id "Device:R") (at 157.48 34.29 0) (unit 1)
     (in_bom yes) (on_board yes)
-    (property "Reference" "R?" (id 0) (at 160.02 33.0199 0)
+    (property "Reference" "R401" (id 0) (at 160.02 33.0199 0)
       (effects (font (size 1.27 1.27)) (justify left))
     )
@@
       (effects (font (size 1.27 1.27)) (justify left))
     )
-    (property "Footprint" "" (id 2) (at 155.702 34.29 90)
+    (property "Footprint" "Resistor_SMD:R_0805_2012Metric_Pad1.20x1.40mm_HandSolder" (id 2) (at 155.702 34.29 90)
       (effects (font (size 1.27 1.27)) hide)
     )
@@
   (symbol (lib_id "power:GND") (at 27.94 54.61 0) (unit 1)
     (in_bom yes) (on_board yes) (fields_autoplaced)
-    (property "Reference" "#PWR?" (id 0) (at 27.94 60.96 0)
+    (property "Reference" "#PWR0401" (id 0) (at 27.94 60.96 0)
       (effects (font (size 1.27 1.27)) hide)
     )
@@
   (symbol (lib_id "Device:R") (at 196.85 34.29 0) (unit 1)
     (in_bom yes) (on_board yes)
-    (property "Reference" "R?" (id 0) (at 199.39 33.0199 0)
+    (property "Reference" "R406" (id 0) (at 199.39 33.0199 0)
       (effects (font (size 1.27 1.27)) (justify left))
     )
@@
       (effects (font (size 1.27 1.27)) (justify left))
     )
-    (property "Footprint" "" (id 2) (at 195.072 34.29 90)
+    (property "Footprint" "Resistor_SMD:R_0805_2012Metric_Pad1.20x1.40mm_HandSolder" (id 2) (at 195.072 34.29 90)
       (effects (font (size 1.27 1.27)) hide)
     )
@@
   (symbol (lib_id "dk_Pushbutton-Switches:GPTS203211B") (at 140.97 49.53 0) (unit 1)
     (in_bom yes) (on_board yes) (fields_autoplaced)
-    (property "Reference" "S?" (id 0) (at 140.97 41.91 0))
+    (property "Reference" "S402" (id 0) (at 140.97 41.91 0))
     (property "Value" "GPTS203211B" (id 1) (at 140.97 44.45 0))
     (property "Footprint" "digikey-footprints:PushButton_12x12mm_THT_GPTS203211B" (id 2) (at 146.05 44.45 0)
@@
   (symbol (lib_id "power:+3.3V") (at 29.21 25.4 0) (unit 1)
     (in_bom yes) (on_board yes) (fields_autoplaced)
-    (property "Reference" "#PWR?" (id 0) (at 29.21 29.21 0)
+    (property "Reference" "#PWR0402" (id 0) (at 29.21 29.21 0)
       (effects (font (size 1.27 1.27)) hide)
     )
@@
   (symbol (lib_id "dk_Pushbutton-Switches:GPTS203211B") (at 140.97 39.37 0) (unit 1)
     (in_bom yes) (on_board yes) (fields_autoplaced)
-    (property "Reference" "S?" (id 0) (at 140.97 31.75 0))
+    (property "Reference" "S401" (id 0) (at 140.97 31.75 0))
     (property "Value" "GPTS203211B" (id 1) (at 140.97 34.29 0))
     (property "Footprint" "digikey-footprints:PushButton_12x12mm_THT_GPTS203211B" (id 2) (at 146.05 34.29 0)
@@
   (symbol (lib_id "power:GND") (at 125.73 86.36 0) (unit 1)
     (in_bom yes) (on_board yes) (fields_autoplaced)
-    (property "Reference" "#PWR?" (id 0) (at 125.73 92.71 0)
+    (property "Reference" "#PWR0403" (id 0) (at 125.73 92.71 0)
       (effects (font (size 1.27 1.27)) hide)
     )
@@
   (symbol (lib_id "power:GND") (at 168.91 24.13 0) (unit 1)
     (in_bom yes) (on_board yes) (fields_autoplaced)
-    (property "Reference" "#PWR?" (id 0) (at 168.91 30.48 0)
+    (property "Reference" "#PWR0404" (id 0) (at 168.91 30.48 0)
       (effects (font (size 1.27 1.27)) hide)
     )
@@
   (symbol (lib_id "Device:R") (at 181.61 34.29 0) (unit 1)
     (in_bom yes) (on_board yes)
-    (property "Reference" "R?" (id 0) (at 184.15 33.0199 0)
+    (property "Reference" "R404" (id 0) (at 184.15 33.0199 0)
       (effects (font (size 1.27 1.27)) (justify left))
     )
@@
       (effects (font (size 1.27 1.27)) (justify left))
     )
-    (property "Footprint" "" (id 2) (at 179.832 34.29 90)
+    (property "Footprint" "Resistor_SMD:R_0805_2012Metric_Pad1.20x1.40mm_HandSolder" (id 2) (at 179.832 34.29 90)
       (effects (font (size 1.27 1.27)) hide)
     )
@@
   (symbol (lib_id "power:+3.3V") (at 180.34 26.67 0) (unit 1)
     (in_bom yes) (on_board yes) (fields_autoplaced)
-    (property "Reference" "#PWR?" (id 0) (at 180.34 30.48 0)
+    (property "Reference" "#PWR0405" (id 0) (at 180.34 30.48 0)
       (effects (font (size 1.27 1.27)) hide)
     )
@@
   (symbol (lib_id "Device:R") (at 187.96 34.29 0) (unit 1)
     (in_bom yes) (on_board yes)
-    (property "Reference" "R?" (id 0) (at 190.5 33.0199 0)
+    (property "Reference" "R405" (id 0) (at 190.5 33.0199 0)
       (effects (font (size 1.27 1.27)) (justify left))
     )
@@
       (effects (font (size 1.27 1.27)) (justify left))
     )
-    (property "Footprint" "" (id 2) (at 186.182 34.29 90)
+    (property "Footprint" "Resistor_SMD:R_0805_2012Metric_Pad1.20x1.40mm_HandSolder" (id 2) (at 186.182 34.29 90)
       (effects (font (size 1.27 1.27)) hide)
     )
@@
   (symbol (lib_id "dk_Pushbutton-Switches:GPTS203211B") (at 140.97 80.01 0) (unit 1)
     (in_bom yes) (on_board yes) (fields_autoplaced)
-    (property "Reference" "S?" (id 0) (at 140.97 72.39 0))
+    (property "Reference" "S405" (id 0) (at 140.97 72.39 0))
     (property "Value" "GPTS203211B" (id 1) (at 140.97 74.93 0))
     (property "Footprint" "digikey-footprints:PushButton_12x12mm_THT_GPTS203211B" (id 2) (at 146.05 74.93 0)
@@
   (symbol (lib_id "Device:R") (at 173.99 34.29 0) (unit 1)
     (in_bom yes) (on_board yes)
-    (property "Reference" "R?" (id 0) (at 176.53 33.0199 0)
+    (property "Reference" "R403" (id 0) (at 176.53 33.0199 0)
       (effects (font (size 1.27 1.27)) (justify left))
     )
@@
       (effects (font (size 1.27 1.27)) (justify left))
     )
-    (property "Footprint" "" (id 2) (at 172.212 34.29 90)
+    (property "Footprint" "Resistor_SMD:R_0805_2012Metric_Pad1.20x1.40mm_HandSolder" (id 2) (at 172.212 34.29 90)
       (effects (font (size 1.27 1.27)) hide)
     )
@@
   (symbol (lib_id "Device:R") (at 165.1 34.29 0) (unit 1)
     (in_bom yes) (on_board yes)
-    (property "Reference" "R?" (id 0) (at 167.64 33.0199 0)
+    (property "Reference" "R402" (id 0) (at 167.64 33.0199 0)
       (effects (font (size 1.27 1.27)) (justify left))
     )
@@
       (effects (font (size 1.27 1.27)) (justify left))
     )
-    (property "Footprint" "" (id 2) (at 163.322 34.29 90)
+    (property "Footprint" "Resistor_SMD:R_0805_2012Metric_Pad1.20x1.40mm_HandSolder" (id 2) (at 163.322 34.29 90)
       (effects (font (size 1.27 1.27)) hide)
     )
@@
   (symbol (lib_id "dk_Pushbutton-Switches:GPTS203211B") (at 140.97 59.69 0) (unit 1)
     (in_bom yes) (on_board yes) (fields_autoplaced)
-    (property "Reference" "S?" (id 0) (at 140.97 52.07 0))
+    (property "Reference" "S403" (id 0) (at 140.97 52.07 0))
     (property "Value" "GPTS203211B" (id 1) (at 140.97 54.61 0))
     (property "Footprint" "digikey-footprints:PushButton_12x12mm_THT_GPTS203211B" (id 2) (at 146.05 54.61 0)
@@
   (symbol (lib_id "dk_Pushbutton-Switches:GPTS203211B") (at 140.97 88.9 0) (unit 1)
     (in_bom yes) (on_board yes) (fields_autoplaced)
-    (property "Reference" "S?" (id 0) (at 140.97 81.28 0))
+    (property "Reference" "S406" (id 0) (at 140.97 81.28 0))
     (property "Value" "GPTS203211B" (id 1) (at 140.97 83.82 0))
     (property "Footprint" "digikey-footprints:PushButton_12x12mm_THT_GPTS203211B" (id 2) (at 146.05 83.82 0)
