File: pcb/onboard_controller.kicad_sch (KiCad schematic)
At the start: 13 parts, among them U401 COM-09032

Commit message: add footprints + fix unnconnected
Connections:
- net bo_button_3: now also S403.2
Changed lines of the file:
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@@
-    (stroke (width 0) (type default) (color 0 0 0 0))
-  )
-  (wire (pts (xy 147.32 59.69) (xy 173.99 59.69))
     (stroke (width 0) (type default) (color 0 0 0 0))
   )
@@
   )
   (wire (pts (xy 181.61 69.85) (xy 205.74 69.85))
+    (stroke (width 0) (type default) (color 0 0 0 0))
+  )
+  (wire (pts (xy 146.05 59.69) (xy 173.99 59.69))
     (stroke (width 0) (type default) (color 0 0 0 0))
   )
@@
       (effects (font (size 1.27 1.27)) hide)
     )
-    (pin "1")
-  )
-  (symbol (lib_id "power:GND") (at 168.91 24.13 0) (unit 1)
-    (in_bom yes) (on_board yes) (fields_autoplaced)
-    (property "Reference" "#PWR0404" (id 0) (at 168.91 30.48 0)
-      (effects (font (size 1.27 1.27)) hide)
-    )
-    (property "Value" "GND" (id 1) (at 168.91 29.21 0))
-    (property "Footprint" "" (id 2) (at 168.91 24.13 0)
-      (effects (font (size 1.27 1.27)) hide)
-    )
-    (property "Datasheet" "" (id 3) (at 168.91 24.13 0)
-      (effects (font (size 1.27 1.27)) hide)
-    )

Commit message: fix joystick
Connections:
- net GND: no longer U401.B2A (SEL-)
- net bo_js_button_1: now also U401.B2A (SEL-); no longer U401.S1 (SHIELD), U401.S2 (SHIELD), U401.S3 (SHIELD), U401.S4 (SHIELD)
- new net: U401.S1 (SHIELD), U401.S2 (SHIELD), U401.S3 (SHIELD), U401.S4 (SHIELD)
Changed lines of the file:
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@@
   (junction (at 181.61 69.85) (diameter 0) (color 0 0 0 0)
   )
-  (junction (at 27.94 48.26) (diameter 0) (color 0 0 0 0)
-  )
   (junction (at 130.81 59.69) (diameter 0) (color 0 0 0 0)
   )
@@
     (stroke (width 0) (type default) (color 0 0 0 0))
   )
-  (wire (pts (xy 27.94 48.26) (xy 27.94 54.61))
+  (wire (pts (xy 27.94 40.64) (xy 27.94 54.61))
     (stroke (width 0) (type default) (color 0 0 0 0))
   )
@@
     (stroke (width 0) (type default) (color 0 0 0 0))
   )
-  (wire (pts (xy 27.94 40.64) (xy 27.94 48.26))
-    (stroke (width 0) (type default) (color 0 0 0 0))
-  )
   (wire (pts (xy 187.96 26.67) (xy 196.85 26.67))
     (stroke (width 0) (type default) (color 0 0 0 0))
@@
   )
   (wire (pts (xy 146.05 80.01) (xy 187.96 80.01))
-    (stroke (width 0) (type default) (color 0 0 0 0))
-  )
-  (wire (pts (xy 27.94 48.26) (xy 43.18 48.26))
     (stroke (width 0) (type default) (color 0 0 0 0))
   )
@@
   (text "Inputs are active low\n" (at 189.23 21.59 0)
     (effects (font (size 1.27 1.27)) (justify left bottom))
-  )
-  (global_label "bo_js_button_1" (shape bidirectional) (at 43.18 53.34 180) (fields_autoplaced)
-    (effects (font (size 1 1)) (justify right))
-    (property "Intersheet References" "${INTERSHEET_REFS}" (id 0) (at 30.1848 53.2775 0)
-      (effects (font (size 1 1)) (justify right) hide)
-    )
   )
   (global_label "bo_js_vert_1" (shape bidirectional) (at 43.18 25.4 180) (fields_autoplaced)
@@
     )
   )
+  (global_label "bo_js_button_1" (shape bidirectional) (at 43.18 48.26 180) (fields_autoplaced)
+    (effects (font (size 1 1)) (justify right))
+    (property "Intersheet References" "${INTERSHEET_REFS}" (id 0) (at 30.1848 48.1975 0)
+      (effects (font (size 1 1)) (justify right) hide)
+    )
+  )
