File: pcb/onboard_controller.kicad_sch (KiCad schematic)
At the start: 13 parts, among them U401 COM-09032

Commit message: fix vias
Parts:
- removed R401, R402, R403, R404, R405, R406: 40k, Resistor_SMD:R_0805_2012Metric_Pad1.20x1.40mm_HandSolder, symbol Device:R
- removed S401, S402, S403, S404, S405, S406: GPTS203211B, digikey-footprints:PushButton_12x12mm_THT_GPTS203211B, symbol dk_Pushbutton-Switches:GPTS203211B
- removed U401: COM-09032, mcu_kicad:XDCR_COM-09032, symbol COM-09032:COM-09032
Connections:
- no-connect marks 1 -> 0
Other:
- note removed: "Inputs are active low"
- note removed: "skal vi koble til push-down på joysticks?"
