File: pcb/pcb.kicad_sch (KiCad schematic)
At the start: 0 parts

Commit message: maybe finished schematic
Other:
- sheet Mcu ports: added DONE, MCU_FPGA_US1_CLK, MCU_FPGA_US1_CS, MCU_FPGA_US1_MISO, MCU_FPGA_US1_MOSI, PROGRAM_B; removed none
- sheet fpga ports: added DONE, FPGA_MCU_EXTRA1, FPGA_MCU_EXTRA2, FPGA_MCU_SPI_CLK, FPGA_MCU_SPI_CS, FPGA_MCU_SPI_SDI, FPGA_MCU_SPI_SDO, PROGRAM_B; removed none

Commit message: everything except crystal
Other:
- sheet Mcu ports: added FPGA_MCU_EXTRA1, FPGA_MCU_EXTRA2; removed none
