File: pcb/fpga_ub.kicad_sch (KiCad schematic)
At the start: 9 parts, among them J1201 Conn_02x07_Top_Bottom, U666 XC7A75T-FTG256

Commit message: is donegst
Connections:
- net FPGA_GPIO_10 is gone; now on net GND: J1201.10 (Pin_10)
- net FPGA_GPIO_9 is gone; now on net +3.3V: J1201.9 (Pin_9)
- net +3.3V: no longer J1201.13 (Pin_13)
- net FPGA_GPIO_1: now also U666.C4 (IO_L12N_T1_MRCC_35)
- net FPGA_GPIO_2: now also U666.D6 (IO_L6P_T0_35); no longer U666.C7 (IO_L5P_T0_AD13P_35)
- net FPGA_GPIO_3: now also U666.C3 (IO_L7P_T1_AD6P_35); no longer U666.C6 (IO_L5N_T0_AD13N_35)
- net FPGA_GPIO_4: now also U666.D4 (IO_L12P_T1_MRCC_35); no longer U666.D6 (IO_L6P_T0_35)
- net FPGA_GPIO_5: now also U666.C2 (IO_L7N_T1_AD6N_35); no longer U666.D5 (IO_L6N_T0_VREF_35)
- net FPGA_GPIO_6: now also U666.D3 (IO_L11N_T1_SRCC_35); no longer U666.C3 (IO_L7P_T1_AD6P_35)
- net FPGA_GPIO_7: now also U666.D1 (IO_L10N_T1_AD15N_35)
- net FPGA_GPIO_8: now also U666.C1 (IO_L9P_T1_DQS_AD7P_35)
- net GND: no longer J1201.14 (Pin_14)
- net FPGA_DEBUG_LED_BLOCK35_1: no longer names the net of U666.H5 (IO_L18P_T2_35)
- net FPGA_DEBUG_LED_BLOCK35_2: no longer names the net of U666.J5 (IO_L19P_T3_35)
- net FPGA_GPIO_11: no longer names the net of J1201.11 (Pin_11)
- net FPGA_GPIO_12: no longer names the net of J1201.12 (Pin_12)
- net FPGA_GPIO_12: no longer U666.E2 (IO_L10P_T1_AD15P_35)
- no-connect marks 39 -> 42
Other:
- note added: "NOTE: H5 and J5 match devboard LEDS in the default constraints file nonono"
- note removed: "NOTE: H5 and J5 match devboard LEDS in the default constraints file"
Changed lines of the file:
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@@
   (no_connect (at 144.78 146.05))
   (no_connect (at 144.78 148.59))
-  (no_connect (at 144.78 151.13))
   (no_connect (at 144.78 153.67))
   (no_connect (at 144.78 156.21))
+  (no_connect (at 200.66 77.47))
   (no_connect (at 43.18 64.77))
   (no_connect (at 43.18 67.31))
-  (no_connect (at 144.78 92.71))
   (no_connect (at 144.78 41.91))
+  (no_connect (at 144.78 72.39))
   (no_connect (at 43.18 41.91))
   (no_connect (at 43.18 44.45))
@@
   (no_connect (at 43.18 57.15))
   (no_connect (at 144.78 95.25))
+  (no_connect (at 144.78 67.31))
+  (no_connect (at 144.78 90.17))
+  (no_connect (at 200.66 72.39))
+  (no_connect (at 144.78 64.77))
   (no_connect (at 144.78 118.11))
   (no_connect (at 144.78 113.03))
-  (no_connect (at 144.78 97.79))
-  (no_connect (at 144.78 100.33))
-  (no_connect (at 144.78 102.87))
   (no_connect (at 144.78 105.41))
   (no_connect (at 144.78 107.95))
@@
   (no_connect (at 43.18 80.01))
   (no_connect (at 43.18 90.17))
-  (no_connect (at 144.78 77.47))
   (no_connect (at 144.78 120.65))
+  (no_connect (at 144.78 135.89))
   (no_connect (at 144.78 158.75))
   (no_connect (at 144.78 161.29))
   (no_connect (at 144.78 163.83))
   (no_connect (at 144.78 166.37))
-  (no_connect (at 144.78 85.09))
+  (no_connect (at 200.66 69.85))
+  (no_connect (at 144.78 130.81))
+  (no_connect (at 200.66 74.93))
   (no_connect (at 144.78 110.49))
   (wire (pts (xy 193.04 29.21) (xy 201.93 29.21))
@@
     (stroke (width 0) (type default) (color 0 0 0 0))
   )
-  (wire (pts (xy 151.13 130.81) (xy 144.78 130.81))
-    (stroke (width 0) (type default) (color 0 0 0 0))
-  )
   (wire (pts (xy 201.93 21.59) (xy 210.82 21.59))
     (stroke (width 0) (type default) (color 0 0 0 0))
@@
     (stroke (width 0) (type default) (color 0 0 0 0))
   )
-  (wire (pts (xy 151.13 135.89) (xy 144.78 135.89))
-    (stroke (width 0) (type default) (color 0 0 0 0))
-  )
   (polyline (pts (xy 171.45 82.55) (xy 171.45 52.07))
     (stroke (width 0) (type default) (color 0 0 0 0))
@@
     (stroke (width 0) (type default) (color 0 0 0 0))
   )
-  (text "NOTE:\nH5 and J5 match devboard LEDS in the default constraints file\n"
+  (text "NOTE:\nH5 and J5 match devboard LEDS in the default constraints file\nnonono"
     (at 162.56 120.65 0)
     (effects (font (size 1.27 1.27)) (justify left bottom))
@@
     (effects (font (size 1.27 1.27)) (justify left bottom))
   )
-  (label "FPGA_GPIO_2" (at 144.78 64.77 0)
-    (effects (font (size 1.27 1.27)) (justify left bottom))
-  )
-  (label "FPGA_GPIO_5" (at 144.78 72.39 0)
-    (effects (font (size 1.27 1.27)) (justify left bottom))
-  )
-  (label "FPGA_GPIO_12" (at 200.66 72.39 0)
-    (effects (font (size 1.27 1.27)) (justify left bottom))
-  )
-  (label "FPGA_GPIO_9" (at 200.66 64.77 0)
-    (effects (font (size 1.27 1.27)) (justify left bottom))
-  )
-  (label "FPGA_GPIO_3" (at 144.78 67.31 0)
-    (effects (font (size 1.27 1.27)) (justify left bottom))
-  )
-  (label "FPGA_GPIO_12" (at 144.78 90.17 0)
+  (label "FPGA_GPIO_7" (at 187.96 77.47 180)
+    (effects (font (size 1.27 1.27)) (justify right bottom))
+  )
+  (label "FPGA_GPIO_2" (at 144.78 69.85 0)
+    (effects (font (size 1.27 1.27)) (justify left bottom))
+  )
+  (label "FPGA_GPIO_8" (at 200.66 62.23 0)
+    (effects (font (size 1.27 1.27)) (justify left bottom))
+  )
+  (label "FPGA_GPIO_4" (at 144.78 100.33 0)
+    (effects (font (size 1.27 1.27)) (justify left bottom))
+  )
+  (label "FPGA_GPIO_7" (at 144.78 92.71 0)
+    (effects (font (size 1.27 1.27)) (justify left bottom))
+  )
+  (label "FPGA_GPIO_6" (at 187.96 74.93 180)
+    (effects (font (size 1.27 1.27)) (justify right bottom))
+  )
+  (label "FPGA_GPIO_5" (at 144.78 77.47 0)
     (effects (font (size 1.27 1.27)) (justify left bottom))
   )
@@
     (effects (font (size 1.27 1.27)) (justify right bottom))
   )
-  (label "FPGA_GPIO_4" (at 144.78 69.85 0)
-    (effects (font (size 1.27 1.27)) (justify left bottom))
-  )
-  (label "FPGA_GPIO_11" (at 200.66 69.85 0)
-    (effects (font (size 1.27 1.27)) (justify left bottom))
-  )
-  (label "FPGA_GPIO_7" (at 187.96 77.47 180)
-    (effects (font (size 1.27 1.27)) (justify right bottom))
+  (label "FPGA_GPIO_8" (at 144.78 85.09 0)
+    (effects (font (size 1.27 1.27)) (justify left bottom))
   )
   (label "FPGA_GPIO_5" (at 187.96 72.39 180)
@@
     (effects (font (size 1.27 1.27)) (justify right bottom))
   )
-  (label "FPGA_GPIO_6" (at 144.78 74.93 0)
-    (effects (font (size 1.27 1.27)) (justify left bottom))
-  )
-  (label "FPGA_GPIO_6" (at 187.96 74.93 180)
-    (effects (font (size 1.27 1.27)) (justify right bottom))
-  )
-  (label "FPGA_GPIO_10" (at 200.66 67.31 0)
-    (effects (font (size 1.27 1.27)) (justify left bottom))
-  )
-  (label "FPGA_GPIO_8" (at 200.66 62.23 0)
+  (label "FPGA_GPIO_3" (at 144.78 74.93 0)
+    (effects (font (size 1.27 1.27)) (justify left bottom))
+  )
+  (label "FPGA_GPIO_6" (at 144.78 97.79 0)
+    (effects (font (size 1.27 1.27)) (justify left bottom))
+  )
+  (label "FPGA_GPIO_1" (at 144.78 102.87 0)
     (effects (font (size 1.27 1.27)) (justify left bottom))
   )
@@
     )
   )
-  (global_label "FPGA_DEBUG_LED_BLOCK35_2" (shape input) (at 151.13 135.89 0) (fields_autoplaced)
-    (effects (font (size 1.27 1.27)) (justify left))
-    (property "Intersheet References" "${INTERSHEET_REFS}" (id 0) (at 181.6645 135.8106 0)
-      (effects (font (size 1.27 1.27)) (justify left) hide)
-    )
-  )
   (global_label "SRAM_A2" (shape bidirectional) (at 43.18 62.23 180) (fields_autoplaced)
     (effects (font (size 1 1)) (justify right))
@@
     (property "Intersheet References" "${INTERSHEET_REFS}" (id 0) (at 151.5848 87.5675 0)
       (effects (font (size 1 1)) (justify left) hide)
-    )
-  )
-  (global_label "FPGA_DEBUG_LED_BLOCK35_1" (shape input) (at 151.13 130.81 0) (fields_autoplaced)
-    (effects (font (size 1.27 1.27)) (justify left))
-    (property "Intersheet References" "${INTERSHEET_REFS}" (id 0) (at 181.6645 130.7306 0)
-      (effects (font (size 1.27 1.27)) (justify left) hide)
     )
   )
@@
     (pin "2")
   )
+  (symbol (lib_id "power:+3.3V") (at 200.66 64.77 270) (unit 1)
+    (in_bom yes) (on_board yes) (fields_autoplaced)
+    (property "Reference" "#PWR0118" (id 0) (at 196.85 64.77 0)
+      (effects (font (size 1.27 1.27)) hide)
+    )
+    (property "Value" "+3.3V" (id 1) (at 204.47 64.7699 90)
+      (effects (font (size 1.27 1.27)) (justify left))
+    )
+    (property "Footprint" "" (id 2) (at 200.66 64.77 0)
+      (effects (font (size 1.27 1.27)) hide)
+    )
+    (property "Datasheet" "" (id 3) (at 200.66 64.77 0)
+      (effects (font (size 1.27 1.27)) hide)
+    )
+    (pin "1")
+  )
   (symbol (lib_id "Device:C") (at 185.42 25.4 0) (unit 1)
     (in_bom yes) (on_board yes)
@@
     (pin "1")
   )
-  (symbol (lib_id "power:+3.3V") (at 200.66 74.93 270) (unit 1)
-    (in_bom yes) (on_board yes) (fields_autoplaced)
-    (property "Reference" "#PWR01202" (id 0) (at 196.85 74.93 0)
-      (effects (font (size 1.27 1.27)) hide)
-    )
-    (property "Value" "+3.3V" (id 1) (at 204.47 74.9299 90)
-      (effects (font (size 1.27 1.27)) (justify left))
-    )
-    (property "Footprint" "" (id 2) (at 200.66 74.93 0)
-      (effects (font (size 1.27 1.27)) hide)
-    )
-    (property "Datasheet" "" (id 3) (at 200.66 74.93 0)
-      (effects (font (size 1.27 1.27)) hide)
-    )
-    (pin "1")
-  )
   (symbol (lib_id "Device:C") (at 238.76 25.4 0) (unit 1)
     (in_bom yes) (on_board yes)
@@
     (pin "2")
   )
+  (symbol (lib_id "power:GND") (at 200.66 67.31 90) (unit 1)
+    (in_bom yes) (on_board yes) (fields_autoplaced)
+    (property "Reference" "#PWR0119" (id 0) (at 207.01 67.31 0)
+      (effects (font (size 1.27 1.27)) hide)
+    )
+    (property "Value" "GND" (id 1) (at 204.47 67.3099 90)
+      (effects (font (size 1.27 1.27)) (justify right))
+    )
+    (property "Footprint" "" (id 2) (at 200.66 67.31 0)
+      (effects (font (size 1.27 1.27)) hide)
+    )
+    (property "Datasheet" "" (id 3) (at 200.66 67.31 0)
+      (effects (font (size 1.27 1.27)) hide)
+    )
+    (pin "1")
+  )
   (symbol (lib_id "Device:C") (at 193.04 25.4 0) (unit 1)
     (in_bom yes) (on_board yes)
@@
     (pin "2")
   )
-  (symbol (lib_id "power:GND") (at 200.66 77.47 90) (unit 1)
-    (in_bom yes) (on_board yes) (fields_autoplaced)
-    (property "Reference" "#PWR01203" (id 0) (at 207.01 77.47 0)
-      (effects (font (size 1.27 1.27)) hide)
-    )
-    (property "Value" "GND" (id 1) (at 204.47 77.4699 90)
-      (effects (font (size 1.27 1.27)) (justify right))
-    )
-    (property "Footprint" "" (id 2) (at 200.66 77.47 0)
-      (effects (font (size 1.27 1.27)) hide)
-    )
-    (property "Datasheet" "" (id 3) (at 200.66 77.47 0)
-      (effects (font (size 1.27 1.27)) hide)
-    )
-    (pin "1")
-  )
   (symbol (lib_id "power:GND") (at 48.26 21.59 270) (unit 1)
