File: pcb/fpga_ua.kicad_sch (KiCad schematic)
At the start: 17 parts, among them U666 XC7A75T-FTG256, Y1101 ECS-2520MV-080-BN-TR

Commit message: is donegst
Connections:
- net FPGA_DEBUG_LED_BLOCK14_1: now also U666.C13 (IO_L12N_T1_MRCC_15); no longer U666.R5 (IO_L23P_T3_A03_D19_14)
- net FPGA_GPIO_9: now also U666.M12 (IO_L6N_T0_D08_VREF_14); no longer U666.L14 (IO_L4P_T0_D04_14)
- net SRAM_A11: now also U666.L14 (IO_L4P_T0_D04_14); no longer U666.K16 (IO_L2N_T0_D03_14)
- net SRAM_A14: now also U666.M14 (IO_L4N_T0_D05_14); no longer U666.K15 (IO_L2P_T0_D02_14)
- net SRAM_A16: now also U666.M15 (IO_L3N_T0_DQS_EMCCLK_14); no longer U666.L15 (IO_L3P_T0_DQS_PUDC_B_14)
- net FPGA_DEBUG_LED_BLOCK35_1: now reaches U666.C12 (IO_L11N_T1_SRCC_15)
- net FPGA_DEBUG_LED_BLOCK35_2: now reaches U666.D13 (IO_L12P_T1_MRCC_15)
- net FPGA_FLASH_D00_IO0: now reaches U666.J13 (IO_L1P_T0_D00_MOSI_14)
- net FPGA_FLASH_D01_IO1: now reaches U666.J14 (IO_L1N_T0_D01_DIN_14)
- net FPGA_FLASH_FCSB_CS: now reaches U666.L12 (IO_L6P_T0_FCS_B_14)
- new net FPGA_FLASH_D02_IO2: U666.K15 (IO_L2P_T0_D02_14)
- new net FPGA_FLASH_D03_IO3: U666.K16 (IO_L2N_T0_D03_14)
- no-connect marks 49 -> 41

Commit message: fix capacitor values and footprints
Parts:
- C1101: footprint Capacitor_SMD:C_0603_1608Metric_Pad1.08x0.95mm_HandSolder -> Capacitor_SMD:C_0805_2012Metric_Pad1.18x1.45mm_HandSolder
Changed lines of the file:
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@@
       (effects (font (size 1.27 1.27)) (justify left))
     )
-    (property "Footprint" "Capacitor_SMD:C_0603_1608Metric_Pad1.08x0.95mm_HandSolder" (id 2) (at 200.3552 123.19 0)
+    (property "Footprint" "Capacitor_SMD:C_0805_2012Metric_Pad1.18x1.45mm_HandSolder" (id 2) (at 200.3552 123.19 0)
       (effects (font (size 1.27 1.27)) hide)
     )
