File: pcb/sram.kicad_sch (KiCad schematic)
At the start: 4 parts

Commit message: add footprints
Parts:
- C701, C702: renamed from C?; footprint (none) -> Capacitor_SMD:C_0603_1608Metric_Pad1.08x0.95mm_HandSolder
- gave numbers to parts that had none: 1
Changed lines of the file:
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@@
   (symbol (lib_id "power:+3.3V") (at 111.76 85.09 0) (unit 1)
     (in_bom yes) (on_board yes) (fields_autoplaced)
-    (property "Reference" "#PWR?" (id 0) (at 111.76 88.9 0)
+    (property "Reference" "#PWR0703" (id 0) (at 111.76 88.9 0)
       (effects (font (size 1.27 1.27)) hide)
     )
@@
   (symbol (lib_id "Device:C") (at 101.6 59.69 180) (unit 1)
     (in_bom yes) (on_board yes) (fields_autoplaced)
-    (property "Reference" "C?" (id 0) (at 105.41 58.4199 0)
+    (property "Reference" "C702" (id 0) (at 105.41 58.4199 0)
       (effects (font (size 1.27 1.27)) (justify right))
     )
@@
       (effects (font (size 1.27 1.27)) (justify right))
     )
-    (property "Footprint" "" (id 2) (at 100.6348 55.88 0)
+    (property "Footprint" "Capacitor_SMD:C_0603_1608Metric_Pad1.08x0.95mm_HandSolder" (id 2) (at 100.6348 55.88 0)
       (effects (font (size 1.27 1.27)) hide)
     )
@@
   (symbol (lib_id "Device:C") (at 87.63 59.69 180) (unit 1)
     (in_bom yes) (on_board yes) (fields_autoplaced)
-    (property "Reference" "C?" (id 0) (at 91.44 58.4199 0)
+    (property "Reference" "C701" (id 0) (at 91.44 58.4199 0)
       (effects (font (size 1.27 1.27)) (justify right))
     )
@@
       (effects (font (size 1.27 1.27)) (justify right))
     )
-    (property "Footprint" "" (id 2) (at 86.6648 55.88 0)
+    (property "Footprint" "Capacitor_SMD:C_0603_1608Metric_Pad1.08x0.95mm_HandSolder" (id 2) (at 86.6648 55.88 0)
       (effects (font (size 1.27 1.27)) hide)
     )
@@
   (symbol (lib_id "sram:AS7C316098A-10TIN") (at 119.38 76.2 0) (unit 2)
     (in_bom yes) (on_board yes) (fields_autoplaced)
-    (property "Reference" "U?" (id 0) (at 153.67 85.09 0)
+    (property "Reference" "U701" (id 0) (at 153.67 85.09 0)
       (effects (font (size 1.524 1.524)) (justify left))
     )
@@
   (symbol (lib_id "power:+3.3V") (at 87.63 52.07 0) (unit 1)
     (in_bom yes) (on_board yes)
-    (property "Reference" "#PWR?" (id 0) (at 87.63 55.88 0)
+    (property "Reference" "#PWR0701" (id 0) (at 87.63 55.88 0)
       (effects (font (size 1.27 1.27)) hide)
     )
@@
   (symbol (lib_id "power:GND") (at 101.6 67.31 0) (unit 1)
     (in_bom yes) (on_board yes) (fields_autoplaced)
-    (property "Reference" "#PWR?" (id 0) (at 101.6 73.66 0)
+    (property "Reference" "#PWR0702" (id 0) (at 101.6 73.66 0)
       (effects (font (size 1.27 1.27)) hide)
     )
@@
   (symbol (lib_id "power:GND") (at 119.38 100.33 0) (unit 1)
     (in_bom yes) (on_board yes) (fields_autoplaced)
-    (property "Reference" "#PWR?" (id 0) (at 119.38 106.68 0)
+    (property "Reference" "#PWR0704" (id 0) (at 119.38 106.68 0)
       (effects (font (size 1.27 1.27)) hide)
     )
@@
   (symbol (lib_id "sram:AS7C316098A-10TIN") (at 33.02 74.93 0) (unit 1)
     (in_bom yes) (on_board yes) (fields_autoplaced)
-    (property "Reference" "U?" (id 0) (at 53.34 63.5 0)
+    (property "Reference" "U701" (id 0) (at 53.34 63.5 0)
       (effects (font (size 1.524 1.524)))
     )

Commit message: make lines between sram and fpga
Connections:
- net SRAM_A0: now also U701.20 (A18); no longer U701.5 (A0)
- net SRAM_A12: now also U701.24 (A14); no longer U701.26 (A12)
- net SRAM_A13: now also U701.23 (A15); no longer U701.25 (A13)
- net SRAM_A14: now also U701.26 (A12); no longer U701.24 (A14)
- net SRAM_A15: now also U701.22 (A16); no longer U701.23 (A15)
- net SRAM_A16: now also U701.25 (A13); no longer U701.22 (A16)
- net SRAM_A18: now also U701.5 (A0); no longer U701.20 (A18)

Commit message: fix capacitor values and footprints
Parts:
- C701, C702: footprint Capacitor_SMD:C_0603_1608Metric_Pad1.08x0.95mm_HandSolder -> Capacitor_SMD:C_0805_2012Metric_Pad1.18x1.45mm_HandSolder
Changed lines of the file:
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@@
       (effects (font (size 1.27 1.27)) (justify right))
     )
-    (property "Footprint" "Capacitor_SMD:C_0603_1608Metric_Pad1.08x0.95mm_HandSolder" (id 2) (at 100.6348 55.88 0)
+    (property "Footprint" "Capacitor_SMD:C_0805_2012Metric_Pad1.18x1.45mm_HandSolder" (id 2) (at 100.6348 55.88 0)
       (effects (font (size 1.27 1.27)) hide)
     )
@@
       (effects (font (size 1.27 1.27)) (justify right))
     )
-    (property "Footprint" "Capacitor_SMD:C_0603_1608Metric_Pad1.08x0.95mm_HandSolder" (id 2) (at 86.6648 55.88 0)
+    (property "Footprint" "Capacitor_SMD:C_0805_2012Metric_Pad1.18x1.45mm_HandSolder" (id 2) (at 86.6648 55.88 0)
       (effects (font (size 1.27 1.27)) hide)
     )
