File: pcb/vga.kicad_sch (KiCad schematic)
At the start: 22 parts, among them J601 DB15_Female_HighDensity

Commit message: fix new vga
Parts:
- J601: footprint vga:618015330923 -> assvga:AHDF15A-KG-TAXB
Changed lines of the file:
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@@
     (property "Reference" "J601" (id 0) (at 127 72.39 0))
     (property "Value" "DB15_Female_HighDensity" (id 1) (at 127 74.93 0))
-    (property "Footprint" "vga:618015330923" (id 2) (at 102.87 85.09 0)
+    (property "Footprint" "assvga:AHDF15A-KG-TAXB" (id 2) (at 102.87 85.09 0)
       (effects (font (size 1.27 1.27)) hide)
     )
